Commit message: fix: 同步脚踝关节训练限位

File: resources/robots/x1/urdf/x1.urdf (robot description, URDF)
Before this commit: robot x1, 58 links, 57 joints
Joints:
- joint left_ankle_pitch_joint: limit lower=-3.14 upper=3.14 effort=80 velocity=10 -> lower=-0.41 upper=0.35 effort=80 velocity=10
- joint left_ankle_roll_joint: limit lower=-3.14 upper=3.14 effort=80 velocity=10 -> lower=-0.64 upper=0.64 effort=80 velocity=10
- joint right_ankle_pitch_joint: limit lower=-3.14 upper=3.14 effort=80 velocity=10 -> lower=-0.41 upper=0.35 effort=80 velocity=10
- joint right_ankle_roll_joint: limit lower=-3.14 upper=3.14 effort=80 velocity=10 -> lower=-0.64 upper=0.64 effort=80 velocity=10
